File: psu_linear_reg.kicad_pcb (KiCad board)
At the start: 2 copper layers, 100 x 40 mm, 26 parts, among them J1 Conn_Coaxial_Power, +V, J2 Conn_Coaxial_Power, -V, J3 Conn_01x10_Pin, J4 Conn_01x10_Pin, J5 Conn_01x10_Pin, J6 Conn_01x10_Pin, J7 Conn_01x05, J8 Conn_01x02, Q3 SI9945BDY-T1-HXY, Q4 SI9945BDY-T1-HXY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

Commit message: rev 1.2. Fixed negative supply nmos protection
Parts:
- removed Q3, Q4: SI9945BDY-T1-HXY, Package_SO:SOP-8_3.76x4.96mm_P1.27mm
- added Q1: AO3400A, Package_TO_SOT_SMD:SOT-23, F.Cu at (145.5, 142.5)
- added Q2: AO3400A, Package_TO_SOT_SMD:SOT-23, F.Cu at (97.0, 133.0)
- J1: value Conn_Coaxial_Power, +V -> Conn_Coaxial_Power
- J2: value Conn_Coaxial_Power, -V -> Conn_Coaxial_Power
- moved R2 10.1 mm to (148.5, 145.5), turned to 0 degrees
- moved R3 6.63 mm to (100.3, 131.0), turned to 0 degrees
Routing:
- net Net-(Q2-S): track 30.0 -> 34.6 mm
- net VEE: track 69.2 -> 72.8 mm
- net Net-(Q2-G): track 4.56 -> 1.99 mm
- net Net-(Q1-G): track 6.88 -> 4.44 mm
- net Net-(Q1-S): track 19.0 -> 19.6 mm
