File: psu_linear_reg.kicad_pcb (KiCad board)
At the start: 2 copper layers, 100 x 40 mm, 26 parts, among them J1 Conn_Coaxial_Power, J2 Conn_Coaxial_Power, J3 Conn_01x10_Pin, J4 Conn_01x10_Pin, J5 Conn_01x10_Pin, J6 Conn_01x10_Pin, J7 Conn_01x05, J8 Conn_01x02, Q1 AO3400A, Q2 AO3400A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

Commit message: V1.3 5-28-25 with -V polarity protection
Other:
- board text added: "J Roth, M Tao, Mueller Group, UC Berkeley rev v1.3: 5-28-25"
- board text removed: "J Roth, M Tao, Mueller Group, UC Berkeley rev v1.2: 1-6-25"
